File: pcb/test.kicad_pcb (KiCad board)
At the start: 2 copper layers, 0 parts

Commit message: Generate serialized net section
Other:
- copper layers 2 -> 0
Changed lines of the file:
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@@
  (page A4)
  (layers
-  (0 F.Cu signal)
-  (31 B.Cu signal)
  )
  (setup
@@
   (uvias_allowed no)
  )
+ (net 0 "")
+ (net 1 +5C)
+ (net 2 GND)
 )
